File: Hardware/relayer_hw.kicad_pcb (KiCad board)
At the start: 4 copper layers, 41 x 88.5 mm, 58 parts, among them J2 AC_OUT, J4 AC_IN, Q1 2N7002, SW1 NRST, SW2 USR_SW, U1 STM32WB55, U2 902-9040, U3 LM1117-3.3, Y1 Crystal, Y2 Crystal_GND23

Commit message: Revisao de hardware
Parts:
- moved L1 11.0 mm to (167.5, 63.5), turned to 180 degrees
- moved Y2 0.56 mm to (149.8, 120.0)
Routing:
- net F: track 21.1 -> 27.6 mm
- net Net-(L1-Pad4): track 13.8 -> 7.86 mm
- net Net-(L1-Pad3): track 14.3 -> 18.4 mm
- net GND: track 19.8 -> 18.5 mm, vias 215 -> 224
- net Net-(U1-Pad25): track 7.19 -> 6.16 mm
- net N: track 77.2 -> 76.3 mm
- added copper zone on In1.Cu, net 3V3
- added copper zone on In2.Cu, net GND
- removed copper zone on VCC, net 3V3
- removed copper zone on GND, net GND
Other:
- outline, holes or cut-outs redrawn
